File: pcb/corrupt.kicad_pcb (KiCad board)
At the start: 2 copper layers, 285 x 94.6 mm, 162 parts, among them J1 USB_C_Receptacle_USB2.0, J2 Conn_01x04_Female, SW1 SW_SPST, SW10 SW_SPST, SW11 SW_SPST, SW12 SW_SPST, SW13 SW_SPST, SW14 SW_SPST, SW15 SW_SPST, SW16 SW_SPST, SW17 SW_SPST, SW18 SW_SPST, SW19 SW_SPST, SW2 SW_SPST, SW20 SW_SPST, SW21 SW_SPST, SW22 SW_SPST, SW23 SW_SPST, SW24 SW_SPST, SW25 SW_SPST, SW26 SW_SPST, SW27 SW_SPST, SW28 SW_SPST, SW29 SW_SPST, SW3 SW_SPST, SW30 SW_SPST, SW31 SW_SPST, SW32 SW_SPST, SW33 SW_SPST, SW34 SW_SPST, SW35 SW_SPST, SW36 SW_SPST, SW37 SW_SPST, SW38 SW_SPST, SW39 SW_SPST, SW4 SW_SPST, SW40 SW_SPST, SW41 SW_SPST, SW42 SW_SPST, SW43 SW_SPST, SW44 SW_SPST, SW45 SW_SPST, SW46 SW_SPST, SW47 SW_SPST, SW48 SW_SPST, SW49 SW_SPST, SW5 SW_SPST, SW50 SW_SPST, SW51 SW_SPST, SW52 SW_SPST, SW53 SW_SPST, SW54 SW_SPST, SW55 SW_SPST, SW56 SW_SPST, SW57 SW_SPST, SW58 SW_SPST, SW59 SW_SPST, SW6 SW_SPST, SW60 SW_SPST, SW61 SW_SPST, SW62 SW_SPST, SW63 SW_SPST, SW64 SW_SPST, SW65 SW_SPST, SW7 SW_SPST, SW8 SW_SPST, SW9 SW_SPST, U1 AMS1117-3.3, U2 SRV05-4-T-P7, U3 STM32F405RGTx, Y1 X322525MOB4SI

Commit message: Update to KiCad 8
Other:
- net class Default removed

Commit message: pcb: v2.0
Parts:
- added D66: LED, LED_SMD:LED_0603_1608Metric, B.Cu at (181.6, 158.2)
- added D67: LED, LED_SMD:LED_0603_1608Metric, B.Cu at (204.3, 158.2)
- added D68: LED, LED_SMD:LED_0603_1608Metric, B.Cu at (63.4, 116.8)
- added D69: LED, LED_SMD:LED_0603_1608Metric, B.Cu at (88.1, 65.7)
- added R1: 330, Resistor_SMD:R_0402_1005Metric, B.Cu at (203.6, 143.3)
- added R10: 1k, Resistor_SMD:R_0402_1005Metric, B.Cu at (64.7, 116.5)
- added R11: 1k, Resistor_SMD:R_0402_1005Metric, B.Cu at (88.4, 67.0)
- added R7: 1k, Resistor_SMD:R_0402_1005Metric, B.Cu at (179.6, 157.7)
- added R8: 10k, Resistor_SMD:R_0402_1005Metric, B.Cu at (164.8, 141.8)
- added R9: 1k, Resistor_SMD:R_0402_1005Metric, B.Cu at (202.3, 157.7)
- R3, R4: value 33 -> 330
- moved R4 37.1 mm to (166.8, 140.8)
- moved R3 37.1 mm to (166.8, 139.8)
- moved C13 0.25 mm to (166.8, 141.8)
Connections:
- J1 pad A8: Net-(J1-PadA8) -> /MCU/SWD
- J1 pad B8: Net-(J1-PadB8) -> /MCU/SWC
- J1 pad S1: Net-(J1-PadS1) -> GND
- J2 pad 3: /MCU/NRST -> Net-(J2-Pin_3)
- U2 pad 1: Net-(U2-Pad1) -> /MCU/SWD
- U2 pad 6: Net-(U2-Pad6) -> /MCU/SWC
- U3 pad 1: Net-(U3-Pad1) -> unconnected-(U3-VBAT-Pad1)
- U3 pad 17: Net-(U3-Pad17) -> /MCU/LED1
- U3 pad 20: Net-(U3-Pad20) -> /MCU/LED2
- U3 pad 21: Net-(U3-Pad21) -> /MCU/LED3
- U3 pad 22: Net-(U3-Pad22) -> /MCU/LED4
- U3 pad 23: Net-(U3-Pad23) -> unconnected-(U3-PA7-Pad23)
- U3 pad 24: Net-(U3-Pad24) -> unconnected-(U3-PC4-Pad24)
- U3 pad 25: Net-(U3-Pad25) -> unconnected-(U3-PC5-Pad25)
- U3 pad 27: Net-(U3-Pad27) -> unconnected-(U3-PB1-Pad27)
- U3 pad 28: Net-(U3-Pad28) -> unconnected-(U3-PB2-Pad28)
- U3 pad 29: Net-(U3-Pad29) -> unconnected-(U3-PB10-Pad29)
- U3 pad 30: Net-(U3-Pad30) -> unconnected-(U3-PB11-Pad30)
- U3 pad 38: Net-(U3-Pad38) -> unconnected-(U3-PC7-Pad38)
- U3 pad 39: Net-(U3-Pad39) -> unconnected-(U3-PC8-Pad39)
- U3 pad 4: Net-(U3-Pad4) -> unconnected-(U3-PC15-Pad4)
- U3 pad 40: Net-(U3-Pad40) -> unconnected-(U3-PC9-Pad40)
- U3 pad 41: Net-(U3-Pad41) -> unconnected-(U3-PA8-Pad41)
- U3 pad 42: Net-(U3-Pad42) -> unconnected-(U3-PA9-Pad42)
- U3 pad 43: Net-(U3-Pad43) -> unconnected-(U3-PA10-Pad43)
- U3 pad 44: Net-(U3-Pad44) -> unconnected-(U3-PA11-Pad44)
- U3 pad 45: Net-(U3-Pad45) -> unconnected-(U3-PA12-Pad45)
- U3 pad 50: Net-(U3-Pad50) -> unconnected-(U3-PA15-Pad50)
- U3 pad 51: Net-(U3-Pad51) -> unconnected-(U3-PC10-Pad51)
- U3 pad 52: Net-(U3-Pad52) -> unconnected-(U3-PC11-Pad52)
- U3 pad 54: Net-(U3-Pad54) -> unconnected-(U3-PD2-Pad54)
- U3 pad 61: Net-(U3-Pad61) -> unconnected-(U3-PB8-Pad61)
Routing:
- net /MCU/SWD: track 24.3 -> 215.3 mm, vias 1 -> 3
- net /MCU/SWC: track 20.3 -> 210.5 mm, vias 1 -> 7
- net /MCU/LED4: track 0.00 -> 150.9 mm, vias 0 -> 4
- net /MCU/LED3: track 0.00 -> 133.7 mm, vias 0 -> 2
- net /Keys/COL3: track 97.2 -> 189.9 mm
- net /Keys/COL6: track 135.9 -> 220.2 mm
- net /Keys/COL12: track 244.4 -> 312.7 mm
- net /Keys/COL1: track 143.7 -> 207.4 mm
- net /Keys/COL9: track 175.5 -> 237.8 mm
- net /Keys/ROW0: track 336.8 -> 390.4 mm
- net /MCU/LED2: track 0.00 -> 51.4 mm, vias 0 -> 2
- net /Keys/COL7: track 138.9 -> 181.0 mm
- net /Keys/COL4: track 82.7 -> 123.5 mm
- net Net-(U3-PA14): track 54.9 -> 16.8 mm
- net Net-(U3-PA13): track 63.2 -> 25.2 mm
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Other:
- outline, holes or cut-outs redrawn
- board text added: "2024-05"
- board text added: "v2.0"
- board text removed: "2021-01"
- board text removed: "v1.0"
