File: pcb/mcu.kicad_sch (KiCad schematic)
At the start: 28 parts, among them J1 USB_C_Receptacle_USB2.0, J2 Conn_01x04_Female, U1 AMS1117-3.3, U2 SRV05-4-T-P7, U3 STM32F405RGTx, Y1 X322525MOB4SI

Commit message: pcb: v2.0
Parts:
- added D66, D67, D68, D69: LED, LED_SMD:LED_0603_1608Metric, symbol Device:LED
- added R1: 330, Resistor_SMD:R_0402_1005Metric, symbol Device:R
- added R10, R11, R7, R9: 1k, Resistor_SMD:R_0402_1005Metric, symbol Device:R
- added R8: 10k, Resistor_SMD:R_0402_1005Metric, symbol Device:R
- C1, C10, C11, C13, C4, C5, C6, C7, C8: LCSC (none) -> C1525
- C12, C14, C15, C2, C3, C9: LCSC (none) -> C19702
- C16, C17: LCSC (none) -> C32949
- R2: LCSC (none) -> C25744
- R3, R4: value 33 -> 330; LCSC (none) -> C25104
- R5, R6: LCSC (none) -> C25905
- U1: LCSC (none) -> C6186
- U2: LCSC (none) -> C7420376
- U3: LCSC (none) -> C15742
- Y1: LCSC (none) -> C9006
Connections:
- net +3V3: now also R8.1
- net GND: now also J1.S1 (SHIELD), D66.1 (K), D67.1 (K), D68.1 (K), D69.1 (K)
- net NRST: now also R1.2, R8.2; no longer J2.3 (Pin_3)
- net SWC: now also J1.B8 (SBU2), U2.6 (IO4)
- net SWD: now also J1.A8 (SBU1), U2.1 (IO1)
- net LED1: now reaches U3.17 (PA3)
- net LED1: now also R7.1
- net LED2: now reaches U3.20 (PA4)
- net LED2: now also R9.1
- net LED3: now reaches U3.21 (PA5)
- net LED3: now also R10.1
- net LED4: now reaches U3.22 (PA6)
- net LED4: now also R11.1
- new net: J2.3 (Pin_3), R1.1
- new net: D69.2 (A), R11.2
- new net: D66.2 (A), R7.2
- new net: D67.2 (A), R9.2
- new net: D68.2 (A), R10.2
